Commit message: Added Front Camera Module

File: catvehicle_basics/catvehicle/urdf/catvehicle_mod.xacro (robot description, xacro)
@@ -117,5 +117,5 @@
         <geometry>
           <!--<mesh filename="package://catvehicle/meshes/ford_escape_no_wheels_2.dae"/>-->
-          <mesh filename="package://catvehicle/meshes/udemy_car_simplified_v2.dae"/>
+          <mesh filename="package://catvehicle/meshes/car_upgraded_camera.dae"/>
           <!--<box size="4.192 ${car_width} ${car_height}"/>-->
         </geometry>
@@ -352,4 +352,30 @@
 </link>
 <!-- Cameras-->
+<joint name="camera_front_joint" type="fixed">
+<origin xyz="0.75 0.0 ${0.725 + camera_box/2 + 1.25}" rpy="0 0 0"/>
+	<axis xyz="0 0 1"/>
+	<parent link="base_link"/>
+	<child link="camera_front_link"/>
+</joint>
+<link name="camera_front_link">
+	<collision>
+	  <origin xyz="0 0 0" rpy="0 0 0"/>
+	  <geometry>
+	   <box size="0.001 0.001 0.001"/>
+	  </geometry>
+	</collision>
+	<visual>
+	  <origin xyz="0 0 0" rpy="0 0 0"/>
+	  <geometry>
+	  <box size="0.001 0.001 0.001"
+/>
+          </geometry>
+	</visual>
+    <inertial>
+      <mass value="1e-5" />
+      <origin xyz="0 0 0" rpy="0 0 0"/>
+      <inertia ixx="1e-6" ixy="0" ixz="0" iyy="1e-6" iyz="0" izz="1e-6" />
+    </inertial>
+</link>
 <!--
 <joint name="camera_right_joint" type="fixed">

Commit message: Added Dedicated car model according to exercises

File: catvehicle_basics/catvehicle/urdf/catvehicle_mod.xacro (robot description, xacro)
@@ -30,6 +30,6 @@
 -->
 <robot name="$(arg roboname)" xmlns:xacro="http://www.ros.org/wiki/xacro">
-  <xacro:arg name="camera_left" default="false"/>
-  <xacro:arg name="camera_right" default="false"/>
+  <xacro:arg name="camera_left" default="true"/>
+  <xacro:arg name="camera_right" default="true"/>
   <xacro:arg name="camera_front" default="true"/>
   <xacro:arg name="camera_back" default="false"/>
@@ -378,7 +378,6 @@
     </inertial>
 </link>
-<!--
 <joint name="camera_right_joint" type="fixed">
-<origin xyz="-0.75 -${car_width/2} ${0.725 + camera_box/2 + 1.25}" rpy="0 0 -${PI/2}"/>
+<origin xyz="1.5 -${car_width/2} ${0.725 + camera_box/2 + 1.25}" rpy="0 0 -${PI/2}"/>
 	<axis xyz="0 0 1"/>
 	<parent link="base_link"/>
@@ -389,5 +388,5 @@
 	  <origin xyz="0 0 0" rpy="0 0 0"/>
 	  <geometry>
-	   <box size="${camera_box} ${camera_box} ${camera_box}"/>
+	   <box size="0.001 0.001 0.001"/>
 	  </geometry>
 	</collision>
@@ -395,5 +394,5 @@
 	  <origin xyz="0 0 0" rpy="0 0 0"/>
 	  <geometry>
-	  <box size="${camera_box} ${camera_box} ${camera_box}"
+	  <box size="0.001 0.001 0.001"
 />
           </geometry>
@@ -406,5 +405,5 @@
 </link>
 <joint name="camera_left_joint" type="fixed">
-<origin xyz="-0.75 ${car_width/2} ${0.725 + camera_box/2 + 1.25}" rpy="0 0 ${PI/2}"/>
+<origin xyz="1.5 ${car_width/2} ${0.725 + camera_box/2 + 1.25}" rpy="0 0 ${PI/2}"/>
 	<axis xyz="0 0 1"/>
 	<parent link="base_link"/>
@@ -415,5 +414,5 @@
 	  <origin xyz="0 0 0" rpy="0 0 0"/>
 	  <geometry>
-	   <box size="${camera_box} ${camera_box} ${camera_box}"/>
+	   <box size="0.001 0.001 0.001"/>
 	  </geometry>
 	</collision>
@@ -421,5 +420,5 @@
 	  <origin xyz="0 0 0" rpy="0 0 0"/>
 	  <geometry>
-	  <box size="${camera_box} ${camera_box} ${camera_box}"
+	  <box size="0.001 0.001 0.001"
 />
           </geometry>
@@ -431,5 +430,4 @@
     </inertial>
 </link>
--->
 <!--
 <joint name="camera_back_joint" type="fixed">

File: catvehicle_basics/catvehicle/urdf/catvehicle_mod_3dlidar.xacro (robot description, xacro)
@@ -35,5 +35,5 @@
   <xacro:arg name="camera_back" default="false"/>
   <xacro:arg name="velodyne_points" default="true"/>
-  <xacro:arg name="front_laser_points" default="true"/>
+  <xacro:arg name="front_laser_points" default="false"/>
   <xacro:property name="PI" value="3.1415926835897931"/>
   <xacro:property name="base_height" value="1.0639"/>
@@ -79,8 +79,4 @@
         <origin xyz="0 0 0" rpy="0 0 ${-PI/2}"/>
   </xacro:property>
-	<!--<xacro:include filename="$(find catvehicle)/urdf/catvehicle.gazebo"/>-->
-    <xacro:if value="${front_laser_points}">
-    	<xacro:include filename="$(find catvehicle)/urdf/catvehicle_front_laser_points.gazebo"/>
-    </xacro:if>
     <xacro:if value="${velodyne_points}">
       <!-- You can pass parameters in order to change the max/min
